File: kicad_project/ITX PiStorm.kicad_pcb (KiCad board)
At the start: 4 copper layers, 170 x 170 mm, 51 parts, among them J2 USB_67298-4090, J201 ATX-20, J3 DB9_Male_MountingHoles, J301 Conn_02x17_Odd_Even, J4 DB9_Male_MountingHoles, J5 HDMI_A_1.4, J6 DB15_Female_HighDensity, Q201 DMG2301L, U201 ST1S10PHR, U202 ADCMP350, U301 74LVC06, U302 74LVC06, U303 74LVC14, U501 LFE5U-85F-6BG381x, U502 W25Q128JVS, U503 MT48LC16M16A2P, U504 MT48LC16M16A2P

Commit message: Wip commit
Parts:
- added G***: LOGO, LOGO, F.Cu at (89.5, 225.0)
- added G***: LOGO, LOGO, F.Cu at (122.0, 212.8)
- added J1: Micro_SD_Card_Det, Connector_Card:microSD_HC_Hirose_DM3D-SF, F.Cu at (137.2, 225.2)
- added U1: TPS2065CDBVT, TPS2065:Texas_Instruments-DBV0005A-0-0-IPC_B, F.Cu at (148.6, 220.7)
Connections:
- Module1 pad 57: unconnected-(Module1-Pad57) -> /CM4 Board/SD_CLK
- Module1 pad 61: unconnected-(Module1-Pad61) -> /CM4 Board/SD_DAT3
- Module1 pad 62: unconnected-(Module1-Pad62) -> /CM4 Board/SD_CMD
- Module1 pad 63: unconnected-(Module1-Pad63) -> /CM4 Board/SD_DAT0
- Module1 pad 67: unconnected-(Module1-Pad67) -> /CM4 Board/SD_DAT1
- Module1 pad 69: unconnected-(Module1-Pad69) -> /CM4 Board/SD_DAT2
Routing:
- net /CM4 Board/SD_DAT2: track 0.00 -> 6.34 mm, vias 0 -> 1
- net /CM4 Board/SD_DAT3: track 0.00 -> 5.74 mm, vias 0 -> 1
- net /CM4 Board/SD_CMD: track 0.00 -> 5.74 mm, vias 0 -> 1
- net /CM4 Board/SD_DAT1: track 0.00 -> 5.56 mm, vias 0 -> 1
- net /CM4 Board/SD_DAT0: track 0.00 -> 5.36 mm, vias 0 -> 1
- net /CM4 Board/SD_CLK: track 0.00 -> 4.20 mm, vias 0 -> 1
- net +5V: track 0.00 -> 3.50 mm, vias 0 -> 4
- net /Memory and Bus Interface/A3: track 30.2 -> 28.3 mm
- net /Memory and Bus Interface/A2: track 31.9 -> 30.3 mm
- net /Memory and Bus Interface/A1: track 29.4 -> 28.0 mm
- net /Memory and Bus Interface/A0: track 31.1 -> 30.0 mm
- net /Memory and Bus Interface/A10: track 28.6 -> 27.7 mm
- net /Memory and Bus Interface/BA1: track 30.3 -> 29.7 mm
- net unconnected-(U501-PadM18): track 0.00 -> 0.40 mm, vias 0 -> 1
- net GND: vias 50 -> 71
