File: kicad_project/cm4.kicad_sch (KiCad schematic)
At the start: 1 part

Commit message: Wip commit
Connections:
- net SD_CLK: now reaches Module1.57 (SD_CLK)
- net SD_DAT3: now reaches Module1.61 (SD_DAT3)
- net SD_CMD: now reaches Module1.62 (SD_CMD)
- net SD_DAT0: now reaches Module1.63 (SD_DAT0)
- net SD_DAT1: now reaches Module1.67 (SD_DAT1)
- net SD_DAT2: now reaches Module1.69 (SD_DAT2)
Changed lines of the file:
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@@
+    (stroke (width 0) (type default) (color 0 0 0 0))
+  )
+  (wire (pts (xy 85.09 111.125) (xy 88.9 111.125))
     (stroke (width 0) (type default) (color 0 0 0 0))
   )
@@
     (stroke (width 0) (type default) (color 0 0 0 0))
   )
+  (wire (pts (xy 88.9 116.205) (xy 85.09 116.205))
+    (stroke (width 0) (type default) (color 0 0 0 0))
+  )
   (wire (pts (xy 24.13 154.305) (xy 22.86 154.305))
     (stroke (width 0) (type default) (color 0 0 0 0))
@@
     (stroke (width 0) (type default) (color 0 0 0 0))
   )
+  (wire (pts (xy 20.955 108.585) (xy 24.13 108.585))
+    (stroke (width 0) (type default) (color 0 0 0 0))
+  )
   (wire (pts (xy 87.63 141.605) (xy 87.63 139.065))
     (stroke (width 0) (type default) (color 0 0 0 0))
@@
     (stroke (width 0) (type default) (color 0 0 0 0))
   )
+  (wire (pts (xy 85.09 118.745) (xy 88.9 118.745))
+    (stroke (width 0) (type default) (color 0 0 0 0))
+  )
   (wire (pts (xy 105.41 131.445) (xy 104.14 131.445))
     (stroke (width 0) (type default) (color 0 0 0 0))
@@
     (stroke (width 0) (type default) (color 0 0 0 0))
   )
+  (wire (pts (xy 85.09 103.505) (xy 88.9 103.505))
+    (stroke (width 0) (type default) (color 0 0 0 0))
+  )
   (wire (pts (xy 166.37 131.445) (xy 167.64 131.445))
     (stroke (width 0) (type default) (color 0 0 0 0))
@@
     (stroke (width 0) (type default) (color 0 0 0 0))
   )
+  (wire (pts (xy 88.9 108.585) (xy 85.09 108.585))
+    (stroke (width 0) (type default) (color 0 0 0 0))
+  )
+  (hierarchical_label "SD_CMD" (shape output) (at 20.955 108.585 180)
+    (effects (font (size 1.27 1.27)) (justify right))
+  )
+  (hierarchical_label "SD_DAT3" (shape bidirectional) (at 88.9 108.585 0)
+    (effects (font (size 1.27 1.27)) (justify left))
+  )
+  (hierarchical_label "SD_DAT0" (shape bidirectional) (at 88.9 111.125 0)
+    (effects (font (size 1.27 1.27)) (justify left))
+  )
+  (hierarchical_label "SD_DAT2" (shape bidirectional) (at 88.9 118.745 0)
+    (effects (font (size 1.27 1.27)) (justify left))
+  )
+  (hierarchical_label "SD_DAT1" (shape bidirectional) (at 88.9 116.205 0)
+    (effects (font (size 1.27 1.27)) (justify left))
+  )
+  (hierarchical_label "SD_CLK" (shape output) (at 88.9 103.505 0)
+    (effects (font (size 1.27 1.27)) (justify left))
+  )
   (symbol (lib_id "CM4IO:ComputeModule4-CM4") (at -3.81 93.345 0) (unit 2)
