File: kicad_project/memory_and_bus.kicad_sch (KiCad schematic)
At the start: 2 parts

Commit message: added bits and pieces: a bit of memory, a bit of 1.1V power
Parts:
- added C501, C502, C503, C504, C505, C506, C507, C508, C509, C510, C511, C512, C513, C514, C515, C516: 100nF, Capacitor_SMD:C_0402_1005Metric, symbol Device:C
- added U502: W25Q128JVS, Package_SO:SOIC-8_5.23x5.23mm_P1.27mm, symbol Memory_Flash:W25Q128JVS
- added U503, U504: MT48LC16M16A2P, Package_SO:TSOP-II-54_22.2x10.16mm_P0.8mm, symbol Memory_RAM:MT48LC16M16A2P
- D501: value (none) -> 1N4148WT; footprint (none) -> Diode_SMD:D_SOD-523
- U501: value (none) -> LFE5U-85F-6BG381x; footprint (none) -> Package_BGA:Lattice_caBGA-381_17.0x17.0mm_Layout20x20_P0.8mm_Ball0.4mm_Pad0.4mm_NSMD
Connections:
- net +3V3: now also U501.T4 (CFG_1), C501.1, C502.1, C503.1, C504.1, C505.1, C506.1, C507.1, C508.1, C509.1, C510.1, C511.1, C512.1, C513.1, C514.1, C515.1, C516.1, U502.8 (VCC), U503.1 (VDD), U503.14 (VDD), U503.27 (VDD), U503.3 (VDDQ), U503.43 (VDDQ), U503.49 (VDDQ), U503.9 (VDDQ), U504.1 (VDD), U504.14 (VDD), U504.27 (VDD), U504.3 (VDDQ), U504.43 (VDDQ), U504.49 (VDDQ), U504.9 (VDDQ)
- net GND: now also C501.2, C502.2, C503.2, C504.2, C505.2, C506.2, C507.2, C508.2, C509.2, C510.2, C511.2, C512.2, C513.2, C514.2, C515.2, C516.2, U502.4 (GND), U503.12 (VSSQ), U503.28 (VSS), U503.41 (VSS), U503.46 (VSSQ), U503.52 (VSSQ), U503.54 (VSS), U503.6 (VSSQ), U504.12 (VSSQ), U504.28 (VSS), U504.41 (VSS), U504.46 (VSSQ), U504.52 (VSSQ), U504.54 (VSS), U504.6 (VSSQ)
- net at U501.R2 (PB15A): now also U502.1 (~{CS})
- net at U501.V2 (PB11A): now also U502.2 (DO(IO1))
- net at U501.W1 (PB9A): now also U502.7 (IO3)
- net at U501.W2 (PB11B): now also U502.5 (DI(IO0))
- net at U501.Y2 (PB9B): now also U502.3 (IO2)
- net ~{CAS}: now reaches U501.M19 (PR47D)
- net ~{CAS}: now also U503.17 (~{CAS}), U504.17 (~{CAS})
- net ~{WE}: now reaches U501.M20 (PR47B)
- net ~{WE}: now also U503.16 (~{WE}), U504.16 (~{WE})
- net ~{CS}: now reaches U501.N19 (PR83A)
- net ~{CS}: now also U503.19 (~{CS}), U504.19 (~{CS})
- net ~{RAS}: now reaches U501.N20 (PR83B)
- net ~{RAS}: now also U503.18 (~{RAS}), U504.18 (~{RAS})
- net BA1: now reaches U501.P19 (PR83C)
- net BA1: now also U503.21 (BA1), U504.21 (BA1)
- net BA0: now reaches U501.P20 (PR86A)
- net BA0: now also U503.20 (BA0), U504.20 (BA0)
- net A10: now reaches U501.R20 (PR86B)
- net A10: now also U503.22 (A10), U504.22 (A10)
- net A0: now reaches U501.T19 (PR89A)
- net A0: now also U503.23 (A0), U504.23 (A0)
- net A1: now reaches U501.T20 (PR86C)
- net A1: now also U503.24 (A1), U504.24 (A1)
- net A2: now reaches U501.U19 (PR89C)
- net A2: now also U503.25 (A2), U504.25 (A2)
- net A3: now reaches U501.U20 (PR86D)
- net A3: now also U503.26 (A3), U504.26 (A3)
- net at U501.U3 (CCLK): now also U502.6 (CLK)
- net +1V2 renamed +1V1
- new net A11: U503.35 (A11), U504.35 (A11)
- new net A12: U503.36 (A12), U504.36 (A12)
- new net A4: U503.29 (A4), U504.29 (A4)
- new net A5: U503.30 (A5), U504.30 (A5)
- new net A6: U503.31 (A6), U504.31 (A6)
- new net A7: U503.32 (A7), U504.32 (A7)
- new net A8: U503.33 (A8), U504.33 (A8)
- new net A9: U503.34 (A9), U504.34 (A9)
- new net CKE: U503.37 (CKE), U504.37 (CKE)
- new net CLK: U503.38 (CLK), U504.38 (CLK)
- new net D0: U503.2 (DQ0)
- new net D1: U503.4 (DQ1)
- new net D10: U503.45 (DQ10)
- new net D11: U503.47 (DQ11)
- new net D12: U503.48 (DQ12)
- new net D13: U503.50 (DQ13)
- new net D14: U503.51 (DQ14)
- new net D15: U503.53 (DQ15)
- new net D16: U504.2 (DQ0)
- new net D17: U504.4 (DQ1)
- new net D18: U504.5 (DQ2)
- new net D19: U504.7 (DQ3)
- new net D2: U503.5 (DQ2)
- new net D20: U504.8 (DQ4)
- new net D21: U504.10 (DQ5)
- new net D22: U504.11 (DQ6)
- new net D23: U504.13 (DQ7)
- new net D24: U504.42 (DQ8)
- new net D25: U504.44 (DQ9)
- new net D26: U504.45 (DQ10)
- new net D27: U504.47 (DQ11)
- new net D28: U504.48 (DQ12)
- new net D29: U504.50 (DQ13)
- new net D3: U503.7 (DQ3)
- new net D30: U504.51 (DQ14)
- new net D31: U504.53 (DQ15)
- new net D4: U503.8 (DQ4)
- new net D5: U503.10 (DQ5)
- new net D6: U503.11 (DQ6)
- new net D7: U503.13 (DQ7)
- new net D8: U503.42 (DQ8)
- new net D9: U503.44 (DQ9)
- new net DQM0: U503.15 (DQML)
- new net DQM1: U503.39 (DQMH)
- new net DQM2: U504.15 (DQML)
- new net DQM3: U504.39 (DQMH)
Other:
- moved on the sheet: D501, U501A, U501B, U501C, U501D, U501E, U501F, U501G, U501H, U501I

Commit message: Wip commit
Parts:
- U503, U504: LCSC (none) -> C26393
Changed lines of the file:
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@@
+      (effects (font (size 1.27 1.27)) hide)
+    )
+    (property "LCSC" "C26393" (id 4) (at 189.23 60.325 0)
       (effects (font (size 1.27 1.27)) hide)
     )
@@
       (effects (font (size 1.27 1.27)) hide)
     )
+    (property "LCSC" "C26393" (id 4) (at 146.05 60.325 0)
+      (effects (font (size 1.27 1.27)) hide)
+    )
